File: 8Selection.kicad_sch (KiCad schematic)
At the start: 0 parts

Commit message: Update everything and keep laying out the i960 features
Use bus wires as much as possible
Other:
- company: (none) -> Joshua Scoggins
Changed lines of the file:
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@@
 (kicad_sch (version 20211123) (generator eeschema)
   (paper "A4")
+  (title_block
+    (date "2022-05-13")
+    (rev "1")
+    (company "Joshua Scoggins")
+  )
   (junction (at 142.494 69.342) (diameter 0) (color 0 0 0 0)
   )
