File: MuxInput.kicad_sch (KiCad schematic)
At the start: 8 parts

Commit message: use the output enable lines on the latches and buffers to do direct logic level conversion
Save some chips in the process.
Parts:
- removed U2, U3, U4, U5: (no value), symbol 74xx:74HC244
- added U? (x4): (no value), symbol 74xx:74LS157
- added U? (x2): (no value), symbol 74xx:74HC02
Connections:
- net GCM4.L0: now also U?.4 (Za)
- net GCM4.L1: now also U?.7 (Zb)
- net GCM4.L10: now also U?.9 (Zc)
- net GCM4.L11: now also U?.12 (Zd)
- net GCM4.L12: now also U?.4 (Za)
- net GCM4.L13: now also U?.7 (Zb)
- net GCM4.L14: now also U?.9 (Zc)
- net GCM4.L15: now also U?.12 (Zd)
- net GCM4.L2: now also U?.9 (Zc)
- net GCM4.L3: now also U?.12 (Zd)
- net GCM4.L4: now also U?.4 (Za)
- net GCM4.L5: now also U?.7 (Zb)
- net GCM4.L6: now also U?.9 (Zc)
- net GCM4.L7: now also U?.12 (Zd)
- net GCM4.L8: now also U?.4 (Za)
- net GCM4.L9: now also U?.7 (Zb)
- net GND: now also U?.8 (GND), U?.8 (GND), U?.8 (GND), U?.8 (GND)
- net VCC: now also U?.16 (VCC), U?.16 (VCC), U?.16 (VCC), U?.16 (VCC)
- net i960.A0: now also U?.2 (I0a)
- net i960.A1: now also U?.5 (I0b)
- net i960.A10: now also U?.11 (I0c)
- net i960.A11: now also U?.14 (I0d)
- net i960.A12: now also U?.2 (I0a)
- net i960.A13: now also U?.5 (I0b)
- net i960.A14: now also U?.11 (I0c)
- net i960.A15: now also U?.14 (I0d)
- net i960.A16: now also U?.3 (I1a)
- net i960.A17: now also U?.6 (I1b)
- net i960.A18: now also U?.10 (I1c)
- net i960.A19: now also U?.13 (I1d)
- net i960.A2: now also U?.11 (I0c)
- net i960.A20: now also U?.3 (I1a)
- net i960.A21: now also U?.6 (I1b)
- net i960.A22: now also U?.10 (I1c)
- net i960.A23: now also U?.13 (I1d)
- net i960.A24: now also U?.3 (I1a)
- net i960.A25: now also U?.6 (I1b)
- net i960.A26: now also U?.10 (I1c)
- net i960.A27: now also U?.13 (I1d)
- net i960.A28: now also U?.3 (I1a)
- net i960.A29: now also U?.6 (I1b)
- net i960.A3: now also U?.14 (I0d)
- net i960.A30: now also U?.10 (I1c)
- net i960.A31: now also U?.13 (I1d)
- net i960.A4: now also U?.2 (I0a)
- net i960.A5: now also U?.5 (I0b)
- net i960.A6: now also U?.11 (I0c)
- net i960.A7: now also U?.14 (I0d)
- net i960.A8: now also U?.2 (I0a)
- net i960.A9: now also U?.5 (I0b)
- new net: U?.10, U?.11, U?.12
- new net GCM4.A0: U?.1 (S), U?.1 (S), U?.1 (S), U?.1 (S)
- new net GCM4.A1: U?.9
- new net GCM4.~{EN}: U?.8
- new net ~{OE}: U?.13, U?.15 (E), U?.15 (E), U?.15 (E), U?.15 (E)
Other:
- moved on the sheet: C2, C3, C4, C5
