File: 8 bit to 4 bit mux.kicad_sch (KiCad schematic)
At the start: 2 parts

Commit message: Keep laying stuff out
Parts:
- gave numbers to parts that had none: 2
Changed lines of the file:
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@@
   (symbol (lib_id "power:GND") (at 128.524 118.364 0) (unit 1)
     (in_bom yes) (on_board yes) (fields_autoplaced)
-    (property "Reference" "#PWR?" (id 0) (at 128.524 124.714 0)
+    (property "Reference" "#PWR0110" (id 0) (at 128.524 124.714 0)
       (effects (font (size 1.27 1.27)) hide)
     )
@@
   (symbol (lib_id "power:VCC") (at 128.524 56.896 0) (unit 1)
     (in_bom yes) (on_board yes) (fields_autoplaced)
-    (property "Reference" "#PWR?" (id 0) (at 128.524 60.706 0)
+    (property "Reference" "#PWR0109" (id 0) (at 128.524 60.706 0)
       (effects (font (size 1.27 1.27)) hide)
     )
@@
   (symbol (lib_id "74xx:74LS157") (at 128.524 86.614 0) (unit 1)
     (in_bom yes) (on_board yes) (fields_autoplaced)
-    (property "Reference" "U?" (id 0) (at 130.5434 65.1342 0)
+    (property "Reference" "U3" (id 0) (at 130.5434 65.1342 0)
       (effects (font (size 1.27 1.27)) (justify left))
     )
@@
   (symbol (lib_id "Device:C") (at 109.728 108.204 0) (unit 1)
     (in_bom yes) (on_board yes) (fields_autoplaced)
-    (property "Reference" "C?" (id 0) (at 112.649 107.3693 0)
+    (property "Reference" "C3" (id 0) (at 112.649 107.3693 0)
       (effects (font (size 1.27 1.27)) (justify left))
     )
