File: Type 2.01 Flattened Board.kicad_pcb (KiCad board)
At the start: 4 copper layers, 170 x 170 mm, 68 parts, among them J1 Conn_02x28_Odd_Even, J2 Conn_01x02, J3 Conn_01x04, J4 Conn_02x03_Odd_Even, J5 Conn_02x03_Odd_Even, J6 Conn_02x28_Odd_Even, U1 74AHC74, U11 74AHC245, U13 74AHC04, U14 ATmega4809-PF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

Commit message: Breakout all unused pins from the management engine
Parts:
- J2: value Conn_01x02 -> Conn_02x18_Odd_Even; footprint Connector_PinHeader_2.54mm:PinHeader_1x02_P2.54mm_Vertical -> Connector_PinHeader_2.54mm:PinHeader_2x18_P2.54mm_Vertical
- U1: value 74AHC74 -> 74LVC1G79; footprint Package_DIP:DIP-14_W7.62mm_Socket -> Package_TO_SOT_SMD:SOT-23-5_HandSoldering
- moved U14 232.0 mm to (102.1, 233.5), turned to 90 degrees
- moved C26 221.5 mm to (113.5, 236.1), turned to 0 degrees
- moved C25 192.5 mm to (123.7, 215.5), turned to 180 degrees
- moved C27 189.5 mm to (144.1, 236.1), turned to 0 degrees
- moved J5 112.6 mm to (103.8, 14.3), turned to 90 degrees
- moved J3 88.3 mm to (191.9, 200.6)
- moved J4 80.0 mm to (155.7, 74.5), turned to 0 degrees
- moved C32 76.1 mm to (153.7, 17.4), turned to 90 degrees
- moved RN1 66.4 mm to (183.5, 46.3)
- moved C31 56.4 mm to (153.7, 47.9), turned to 90 degrees
- moved U1 55.1 mm to (156.2, 30.2), turned to 90 degrees
- moved U16 52.2 mm to (150.8, 59.3), turned to 180 degrees
- moved C1 47.8 mm to (156.2, 26.6), turned to 0 degrees
- moved C30 35.0 mm to (132.9, 37.7), turned to -90 degrees
- moved C29 24.8 mm to (106.2, 130.5)
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Connections:
- C10 pad 1: VCC -> +5V
- C14 pad 1: VCC -> +5V
- C15 pad 1: VCC -> +5V
- C19 pad 1: VCC -> +5V
- C2 pad 1: VCC -> +5V
- C3 pad 1: VCC -> +5V
- C35 pad 1: VCC -> +5V
- C36 pad 1: VCC -> +5V
- C9 pad 1: VCC -> +5V
- J2 pad 1: /i960/CTRL07/IN6 -> /i960/PIC.PA6
- J2 pad 2: /i960/CTRL07/IN7 -> /i960/PIC.PA6
- RN1 pad 5: /i960/PU0 -> unconnected-(RN1-Pad5)
- RN1 pad 6: /i960/PU1 -> unconnected-(RN1-Pad6)
- RN1 pad 7: /i960/PU2 -> unconnected-(RN1-Pad7)
- RN1 pad 8: /i960/PU3 -> unconnected-(RN1-Pad8)
- U1 pad 1: (no net) -> /i960/FAIL_SIG
- U1 pad 2: (no net) -> /i960.CLK
- U1 pad 3: (no net) -> GND
- U1 pad 4: (no net) -> /i960/~{ME_FAIL_IN}
- U1 pad 5: (no net) -> +5V
- U11 pad 1: VCC -> +5V
- U11 pad 20: VCC -> +5V
- U11 pad 8: /i960/CTRL07/IN6 -> GND
- U11 pad 9: /i960/CTRL07/IN7 -> GND
- U13 pad 1: Net-(U17-Pad4) -> /i960/K0
- U13 pad 3: Net-(U17-Pad12) -> /i960/K3
- U17 pad 11: /i960/INT2_OUT -> /i960/INT1_OUT
- U17 pad 12: Net-(U17-Pad12) -> /i960/i960.INT2
- U17 pad 14: /i960/INT3_OUT -> /i960/INT2_OUT
- U17 pad 2: /i960/INT0_OUT -> /i960/INT3_OUT
- U17 pad 4: Net-(U17-Pad4) -> /i960/K3
- U17 pad 5: /i960/INT1_OUT -> /i960/INT0_OUT
- U17 pad 7: /i960/i960.INT1 -> /i960/K0
- U17 pad 9: /i960/i960.INT2 -> /i960/i960.INT1
- U18 pad 20: VCC -> +5V
- U19 pad 20: VCC -> +5V
- U2 pad 1: VCC -> +5V
- U2 pad 20: VCC -> +5V
- U3 pad 16: VCC -> +5V
- U3 pad 6: VCC -> +5V
- U4 pad 1: VCC -> +5V
- U4 pad 20: VCC -> +5V
- U6 pad 1: VCC -> +5V
- U6 pad 20: VCC -> +5V
- U7 pad 23: VCC -> +5V
- U7 pad 24: VCC -> +5V
- U8 pad 23: VCC -> +5V
- U8 pad 24: VCC -> +5V
- XA1 pad IORF: VCC -> +5V
- XA2 pad IORF: VCC -> +5V

Commit message: Start routing
Parts:
- RN1: value R_Network12 -> R_Network04; footprint Resistor_THT:R_Array_SIP13 -> Resistor_THT:R_Array_SIP5
- moved RN1 156.1 mm to (66.2, 149.3), turned to 0 degrees
- moved C32 151.6 mm to (61.5, 137.8), turned to -90 degrees
- moved J4 142.8 mm to (14.2, 93.8), turned to 180 degrees
- moved C1 141.8 mm to (59.0, 129.8), turned to 180 degrees
- moved U1 136.7 mm to (59.0, 126.3), turned to -90 degrees
- moved C31 109.5 mm to (61.5, 107.2), turned to -90 degrees
- moved J5 108.3 mm to (14.1, 75.0), turned to 180 degrees
- moved J3 100.1 mm to (142.6, 113.5), turned to 0 degrees
- moved C30 94.4 mm to (82.3, 117.4), turned to 90 degrees
- moved U16 93.8 mm to (64.4, 95.8), turned to 0 degrees
- moved C27 85.9 mm to (139.3, 150.4)
- moved C25 85.9 mm to (118.9, 129.8)
- moved C26 85.9 mm to (108.7, 150.4)
- moved U14 85.9 mm to (97.4, 147.7)
- moved C8 37.7 mm to (105.5, 47.2), turned to 180 degrees
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Connections:
- U4 pad 13: /GCM4.HLDA -> /GCM4.USART_PIC_RX
- U4 pad 14: /GCM4.USART_PIC_RX -> /GCM4.HLDA
- U4 pad 16: /GCM4.~{DO_CYCLE} -> /GCM4.~{BURST_LAST}
- U4 pad 17: /GCM4.~{IN_TRANSACTION} -> /GCM4.~{DO_CYCLE}
- U4 pad 18: /GCM4.~{BURST_LAST} -> /GCM4.~{IN_TRANSACTION}
- U4 pad 2: /i960/i960.~{BURST_LAST} -> /i960/i960.~{IN_TRANSACTION}
- U4 pad 3: /i960/i960.~{IN_TRANSACTION} -> /i960/i960.~{DO_CYCLE}
- U4 pad 4: /i960/i960.~{DO_CYCLE} -> /i960/i960.~{BURST_LAST}
- U4 pad 6: /i960/PIC.TX -> /i960/i960.HLDA
- U4 pad 7: /i960/i960.HLDA -> /i960/PIC.TX
- XA1 pad D10: /GCM4.~{BOOT_SUCCESSFUL} -> /GCM4.~{DO_CYCLE}
- XA1 pad D11: /GCM4.~{BURST_LAST} -> /GCM4.~{IN_TRANSACTION}
- XA1 pad D12: /GCM4.~{DO_CYCLE} -> /GCM4.~{FEATHER_INT1}
- XA1 pad D13: /GCM4.~{IN_TRANSACTION} -> /GCM4.~{FEATHER_INT0}
- XA1 pad D8: /GCM4.~{FEATHER_INT1} -> /GCM4.~{BOOT_SUCCESSFUL}
- XA1 pad D9: /GCM4.~{FEATHER_INT0} -> /GCM4.~{BURST_LAST}
Routing:
- net /AREF: track 0.00 -> 223.6 mm
- net /SCL: track 0.00 -> 222.5 mm
- net /SDA: track 0.00 -> 222.4 mm
- net /GCM4.USART_PIC_RX: track 0.00 -> 30.4 mm
- net GND: track 0.00 -> 18.4 mm
- net +5V: track 0.00 -> 11.6 mm, vias 0 -> 2
- net /GCM4.HLDA: track 0.00 -> 9.37 mm
- net /GCM4.~{BOOT_SUCCESSFUL}: track 0.00 -> 8.21 mm
- net /GCM4.~{BURST_LAST}: track 0.00 -> 7.68 mm
- net /GCM4.~{IN_TRANSACTION}: track 0.00 -> 7.51 mm
- net /GCM4.~{DO_CYCLE}: track 0.00 -> 7.25 mm
