File: i960ToGCM4LBus245.kicad_sch (KiCad schematic)
At the start: 2 parts

Commit message: Design simplification
Parts:
- gave numbers to parts that had none: 2
Changed lines of the file:
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@@
   (symbol (lib_id "74xx:74HC245") (at 132.334 73.152 0) (unit 1)
     (in_bom yes) (on_board yes) (fields_autoplaced)
-    (property "Reference" "U?" (id 0) (at 134.3534 54.2122 0)
+    (property "Reference" "U6" (id 0) (at 134.3534 54.2122 0)
       (effects (font (size 1.27 1.27)) (justify left))
     )
@@
   (symbol (lib_id "power:VCC") (at 132.334 44.196 0) (unit 1)
     (in_bom yes) (on_board yes) (fields_autoplaced)
-    (property "Reference" "#PWR?" (id 0) (at 132.334 48.006 0)
+    (property "Reference" "#PWR013" (id 0) (at 132.334 48.006 0)
       (effects (font (size 1.27 1.27)) hide)
     )
@@
   (symbol (lib_id "power:GND") (at 132.334 104.394 0) (unit 1)
     (in_bom yes) (on_board yes) (fields_autoplaced)
-    (property "Reference" "#PWR?" (id 0) (at 132.334 110.744 0)
+    (property "Reference" "#PWR014" (id 0) (at 132.334 110.744 0)
       (effects (font (size 1.27 1.27)) hide)
     )
@@
   (symbol (lib_id "Device:C") (at 155.448 92.202 0) (unit 1)
     (in_bom yes) (on_board yes) (fields_autoplaced)
-    (property "Reference" "C?" (id 0) (at 158.369 91.3673 0)
+    (property "Reference" "C14" (id 0) (at 158.369 91.3673 0)
       (effects (font (size 1.27 1.27)) (justify left))
     )

Commit message: Correct the feather symbol and breakouts
Also fix the VCC pin being bound to +5V for some reason. Use VCCIO
instead
Connections:
- net VCC renamed VCCIO
Changed lines of the file:
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@@
     (pin "9")
-  )
-  (symbol (lib_id "power:VCC") (at 132.334 44.196 0) (unit 1)
-    (in_bom yes) (on_board yes) (fields_autoplaced)
-    (property "Reference" "#PWR013" (id 0) (at 132.334 48.006 0)
-      (effects (font (size 1.27 1.27)) hide)
-    )
-    (property "Value" "" (id 1) (at 132.334 40.6202 0))
-    (property "Footprint" "" (id 2) (at 132.334 44.196 0)
-      (effects (font (size 1.27 1.27)) hide)
-    )
-    (property "Datasheet" "" (id 3) (at 132.334 44.196 0)
-      (effects (font (size 1.27 1.27)) hide)
-    )
-    (pin "1")
   )
   (symbol (lib_id "power:GND") (at 132.334 104.394 0) (unit 1)
@@
     (pin "1")
   )
+  (symbol (lib_id "SparkFun-PowerSymbols:VCCIO") (at 132.334 44.196 0) (unit 1)
+    (in_bom yes) (on_board yes) (fields_autoplaced)
+    (property "Reference" "#SUPPLY0111" (id 0) (at 133.604 44.196 0)
+      (effects (font (size 1.143 1.143)) (justify left bottom) hide)
+    )
+    (property "Value" "" (id 1) (at 132.334 37.9143 0)
+      (effects (font (size 1.143 1.143)))
+    )
+    (property "Footprint" "" (id 2) (at 132.334 40.5653 0)
+      (effects (font (size 1.524 1.524)))
+    )
+    (property "Datasheet" "" (id 3) (at 132.334 44.196 0)
+      (effects (font (size 1.524 1.524)) hide)
+    )
+    (pin "~")
+  )
   (symbol (lib_id "Device:C") (at 155.448 92.202 0) (unit 1)

Commit message: Fix naming + more features
Parts:
- C14: value (none) -> 0.1uF; footprint (none) -> Capacitor_SMD:C_0805_2012Metric_Pad1.18x1.45mm_HandSolder
- U6: value (none) -> 74AHC245; footprint (none) -> Package_SO:SOIC-20W_7.5x12.8mm_P1.27mm
Changed lines of the file:
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@@
       (effects (font (size 1.27 1.27)) (justify left))
     )
-    (property "Value" "" (id 1) (at 134.3534 56.7491 0)
+    (property "Value" "74AHC245" (id 1) (at 134.3534 56.7491 0)
       (effects (font (size 1.27 1.27)) (justify left))
     )
-    (property "Footprint" "" (id 2) (at 132.334 73.152 0)
+    (property "Footprint" "Package_SO:SOIC-20W_7.5x12.8mm_P1.27mm" (id 2) (at 132.334 73.152 0)
       (effects (font (size 1.27 1.27)) hide)
     )
@@
       (effects (font (size 1.27 1.27)) hide)
     )
-    (property "Value" "" (id 1) (at 132.334 108.8374 0))
+    (property "Value" "GND" (id 1) (at 132.334 108.8374 0))
     (property "Footprint" "" (id 2) (at 132.334 104.394 0)
       (effects (font (size 1.27 1.27)) hide)
@@
   (symbol (lib_id "SparkFun-PowerSymbols:VCCIO") (at 132.334 44.196 0) (unit 1)
     (in_bom yes) (on_board yes) (fields_autoplaced)
-    (property "Reference" "#SUPPLY0111" (id 0) (at 133.604 44.196 0)
+    (property "Reference" "#SUPPLY0110" (id 0) (at 133.604 44.196 0)
       (effects (font (size 1.143 1.143)) (justify left bottom) hide)
     )
-    (property "Value" "" (id 1) (at 132.334 37.9143 0)
+    (property "Value" "VCCIO" (id 1) (at 132.334 37.9143 0)
       (effects (font (size 1.143 1.143)))
     )
-    (property "Footprint" "" (id 2) (at 132.334 40.5653 0)
+    (property "Footprint" "XXX-00000" (id 2) (at 132.334 40.5653 0)
       (effects (font (size 1.524 1.524)))
     )
@@
       (effects (font (size 1.27 1.27)) (justify left))
     )
-    (property "Value" "" (id 1) (at 158.369 93.9042 0)
+    (property "Value" "0.1uF" (id 1) (at 158.369 93.9042 0)
       (effects (font (size 1.27 1.27)) (justify left))
     )
-    (property "Footprint" "" (id 2) (at 156.4132 96.012 0)
+    (property "Footprint" "Capacitor_SMD:C_0805_2012Metric_Pad1.18x1.45mm_HandSolder" (id 2) (at 156.4132 96.012 0)
       (effects (font (size 1.27 1.27)) hide)
     )
